File: Hidrometro lacrador.kicad_pcb (KiCad board)
At the start: 2 copper layers, 4 parts, among them U1 ESP32-WROOM-V1

Commit message: Finalização do circuito e da PCB
Parts:
- added LED-ON1: LED, TerminalBlock:TerminalBlock_Altech_AK300-2_P5.00mm, F.Cu at (31.1, 42.4)
- added R1: 330, Resistor_THT:R_Axial_DIN0414_L11.9mm_D4.5mm_P20.32mm_Horizontal, F.Cu at (74.6, 61.1)
- moved Alimentação1 16.3 mm to (32.4, 84.4), turned to 0 degrees
- moved SensorDeFluxo1 13.0 mm to (65.0, 84.3), turned to 0 degrees
- moved DisplayLCD-I2C1 0.79 mm to (43.7, 84.4)
Connections:
- DisplayLCD-I2C1 pad 3: unconnected-(DisplayLCD-I2C1-Pin_3-Pad3) -> I2C_SDA
- DisplayLCD-I2C1 pad 4: unconnected-(DisplayLCD-I2C1-Pin_4-Pad4) -> I2C_SCL
- SensorDeFluxo1 pad 1: +5V -> +3.3V
- SensorDeFluxo1 pad 2: unconnected-(SensorDeFluxo1-Pin_2-Pad2) -> GPIO-04
- U1 pad 20: unconnected-(U1-GPI21/I2C_SDA-Pad20) -> I2C_SCL
- U1 pad 21: unconnected-(U1-GPI19/VSPI_MISO-Pad21) -> I2C_SDA
- U1 pad 26: unconnected-(U1-GPIO04/ADC10-Pad26) -> GPIO-04
- U1 pad 30: unconnected-(U1-3.3V-Pad30) -> +3.3V
Routing:
- net GND: track 54.1 -> 128.1 mm
- net Net-(LED-ON1-A): track 0.00 -> 66.5 mm
- net I2C_SCL: track 0.00 -> 61.9 mm
- net +5V: track 190.3 -> 135.6 mm
- net I2C_SDA: track 0.00 -> 43.0 mm
- net GPIO-04: track 0.00 -> 26.7 mm
- net +3.3V: track 0.00 -> 18.4 mm
Other:
- board outline added: 59.1 x 69 mm

Commit message: mudança das portas do display LCD
Parts:
- renumbered LED-ON1 to LED-ON/OFF1
Connections:
- U1 pad 17: unconnected-(U1-GPI22/I2C_SCL-Pad17) -> I2C_SCL
- U1 pad 20: I2C_SCL -> I2C_SDA
- U1 pad 21: I2C_SDA -> unconnected-(U1-GPI19/VSPI_MISO-Pad21)
Routing:
- net I2C_SCL: track 61.9 -> 70.0 mm
- net I2C_SDA: track 43.0 -> 46.4 mm
Changed lines of the file:
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@@
 	(net 7 "I2C_SDA")
 	(net 8 "+5V")
-	(net 9 "unconnected-(U1-GPI22{slash}I2C_SCL-Pad17)")
+	(net 9 "Net-(LED-ON/OFF1-A)")
 	(net 10 "unconnected-(U1-GPIO39{slash}ADC3-Pad3)")
 	(net 11 "unconnected-(U1-GPIO14{slash}ADC16{slash}TOUCH6-Pad11)")
@@
 	(net 28 "GPIO-04")
 	(net 29 "unconnected-(U1-GPIO02{slash}ADC13-Pad27)")
-	(net 30 "Net-(LED-ON1-A)")
+	(net 30 "unconnected-(U1-GPI19{slash}VSPI_MISO-Pad21)")
 	(footprint "TerminalBlock:TerminalBlock_Altech_AK300-2_P5.00mm"
 		(layer "F.Cu")
@@
 		(descr "Altech AK300 terminal block, pitch 5.0mm, 45 degree angled, see http://www.mouser.com/ds/2/16/PCBMETRC-24178.pdf")
 		(tags "Altech AK300 terminal block pitch 5.0mm")
-		(property "Reference" "LED-ON1"
+		(property "Reference" "LED-ON/OFF1"
 			(at -1.92 -6.99 90)
 			(layer "F.SilkS")
@@
 				(font
 					(size 1.27 1.27)
+					(thickness 0.15)
 				)
 			)
@@
 				(font
 					(size 1.27 1.27)
+					(thickness 0.15)
 				)
 			)
@@
 				(font
 					(size 1.27 1.27)
+					(thickness 0.15)
 				)
 			)
 		)
 		(property ki_fp_filters "LED* LED_SMD:* LED_THT:*")
-		(sheetname "Root")
+		(sheetname "Raiz")
 		(sheetfile "Hidrometro lacrador.kicad_sch")
 		(attr through_hole)
@@
 			(layers "*.Cu" "*.Mask")
 			(remove_unused_layers no)
-			(net 30 "Net-(LED-ON1-A)")
+			(net 9 "Net-(LED-ON/OFF1-A)")
 			(pinfunction "A")
 			(pintype "passive")
@@
 		(tags "Altech AK300 terminal block pitch 5.0mm")
 		(property "Reference" "SensorDeFluxo1"
-			(at 5 -7.1 360)
+			(at 5 -7.1 0)
 			(layer "F.SilkS")
 			(effects
@@
 		)
 		(property "Value" "Screw_Terminal_01x03"
-			(at 4.95 7.3 360)
+			(at 4.95 7.3 0)
 			(layer "F.Fab")
 			(effects
@@
 				(font
 					(size 1.27 1.27)
+					(thickness 0.15)
 				)
 			)
@@
 				(font
 					(size 1.27 1.27)
+					(thickness 0.15)
 				)
 			)
@@
 				(font
 					(size 1.27 1.27)
+					(thickness 0.15)
 				)
 			)
 		)
 		(property ki_fp_filters "TerminalBlock*:*")
-		(sheetname "Root")
+		(sheetname "Raiz")
 		(sheetfile "Hidrometro lacrador.kicad_sch")
 		(attr through_hole)
@@
 		)
 		(fp_text user "${REFERENCE}"
-			(at 5 -2 360)
+			(at 5 -2 0)
 			(layer "F.Fab")
 			(effects
@@
 				(font
 					(size 1.27 1.27)
+					(thickness 0.15)
 				)
 			)
@@
 				(font
 					(size 1.27 1.27)
+					(thickness 0.15)
 				)
 			)
@@
 				(font
 					(size 1.27 1.27)
+					(thickness 0.15)
 				)
 			)
 		)
 		(property ki_fp_filters "TerminalBlock*:*")
-		(sheetname "Root")
+		(sheetname "Raiz")
 		(sheetfile "Hidrometro lacrador.kicad_sch")
 		(attr through_hole)
@@
 		(tags "Altech AK300 terminal block pitch 5.0mm")
 		(property "Reference" "Alimentação1"
-			(at -1.92 -6.99 360)
+			(at -1.92 -6.99 0)
 			(layer "F.SilkS")
 			(effects
@@
 		)
 		(property "Value" "Screw_Terminal_01x02"
-			(at 2.78 7.75 360)
+			(at 2.78 7.75 0)
 			(layer "F.Fab")
 			(effects
@@
 				(font
 					(size 1.27 1.27)
+					(thickness 0.15)
 				)
 			)
@@
 				(font
 					(size 1.27 1.27)
+					(thickness 0.15)
 				)
 			)
@@
 				(font
 					(size 1.27 1.27)
+					(thickness 0.15)
 				)
 			)
 		)
 		(property ki_fp_filters "TerminalBlock*:*")
-		(sheetname "Root")
+		(sheetname "Raiz")
 		(sheetfile "Hidrometro lacrador.kicad_sch")
 		(attr through_hole)
@@
 		)
 		(fp_text user "${REFERENCE}"
-			(at 2.5 -2 360)
+			(at 2.5 -2 0)
 			(layer "F.Fab")
 			(effects
@@
 		(tags "Resistor Axial_DIN0414 series Axial Horizontal pin pitch 20.32mm 2W length 11.9mm diameter 4.5mm")
 		(property "Reference" "R1"
-			(at 10.16 -3.37 270)
+			(at 10.16 -3.37 -90)
 			(layer "F.SilkS")
 			(effects
@@
 		)
 		(property "Value" "330"
-			(at 10.16 3.37 270)
+			(at 10.16 3.37 -90)
 			(layer "F.Fab")
 			(effects
@@
 				(font
 					(size 1.27 1.27)
+					(thickness 0.15)
 				)
 			)
@@
 				(font
 					(size 1.27 1.27)
+					(thickness 0.15)
 				)
 			)
@@
 				(font
 					(size 1.27 1.27)
+					(thickness 0.15)
 				)
 			)
 		)
 		(property ki_fp_filters "R_*")
-		(sheetname "Root")
+		(sheetname "Raiz")
 		(sheetfile "Hidrometro lacrador.kicad_sch")
 		(attr through_hole)
@@
 		)
 		(fp_text user "${REFERENCE}"
-			(at 10.16 0 270)
+			(at 10.16 0 -90)
 			(layer "F.Fab")
 			(effects
@@
 			(layers "*.Cu" "*.Mask")
 			(remove_unused_layers no)
-			(net 30 "Net-(LED-ON1-A)")
+			(net 9 "Net-(LED-ON/OFF1-A)")
 			(pintype "passive")
 		)
@@
 			)
 		)
-		(sheetname "Root")
+		(sheetname "Raiz")
 		(sheetfile "Hidrometro lacrador.kicad_sch")
 		(attr smd)
@@
 			(layers "*.Cu" "*.Mask")
 			(remove_unused_layers no)
-			(net 9 "unconnected-(U1-GPI22{slash}I2C_SCL-Pad17)")
+			(net 5 "I2C_SCL")
 			(pinfunction "GPI22/I2C_SCL")
 			(pintype "bidirectional")
@@
 			(layers "*.Cu" "*.Mask")
 			(remove_unused_layers no)
-			(net 5 "I2C_SCL")
+			(net 7 "I2C_SDA")
 			(pinfunction "GPI21/I2C_SDA")
 			(pintype "bidirectional")
@@
 			(layers "*.Cu" "*.Mask")
 			(remove_unused_layers no)
-			(net 7 "I2C_SDA")
+			(net 30 "unconnected-(U1-GPI19{slash}VSPI_MISO-Pad21)")
 			(pinfunction "GPI19/VSPI_MISO")
 			(pintype "bidirectional")
@@
 	)
 	(segment
-		(start 50.8508 86.6394)
-		(end 50.8508 55.6768)
+		(start 58.6918 84.3534)
+		(end 58.6918 87.5106)
 		(width 1.2)
 		(layer "B.Cu")
@@
 	)
 	(segment
-		(start 60.75 45.7776)
-		(end 65.3364 45.7776)
+		(start 52.8828 88.6714)
+		(end 50.8508 86.6394)
 		(width 1.2)
 		(layer "B.Cu")
@@
 	)
 	(segment
-		(start 58.6918 87.5106)
-		(end 57.531 88.6714)
+		(start 59.8424 38.1576)
+		(end 65.3364 38.1576)
 		(width 1.2)
 		(layer "B.Cu")
@@
 	)
 	(segment
-		(start 50.8508 55.6768)
-		(end 60.75 45.7776)
+		(start 58.6918 87.5106)
+		(end 57.531 88.6714)
 		(width 1.2)
 		(layer "B.Cu")
@@
 	)
 	(segment
-		(start 57.531 88.6714)
-		(end 52.8828 88.6714)
+		(start 50.8508 86.6394)
+		(end 50.8508 47.1492)
 		(width 1.2)
 		(layer "B.Cu")
@@
 	)
 	(segment
-		(start 58.6918 84.3534)
-		(end 58.6918 87.5106)
+		(start 50.8508 47.1492)
+		(end 59.8424 38.1576)
 		(width 1.2)
 		(layer "B.Cu")
@@
 	)
 	(segment
-		(start 52.8828 88.6714)
-		(end 50.8508 86.6394)
+		(start 57.531 88.6714)
+		(end 52.8828 88.6714)
 		(width 1.2)
 		(layer "B.Cu")
@@
 	)
 	(segment
-		(start 53.6918 56.2648)
+		(start 53.6918 52.3082)
 		(end 53.6918 84.3534)
 		(width 1.2)
@@
 	)
 	(segment
-		(start 65.3364 48.3176)
-		(end 61.639 48.3176)
+		(start 60.2224 45.7776)
+		(end 53.6918 52.3082)
 		(width 1.2)
 		(layer "B.Cu")
@@
 	)
 	(segment
-		(start 61.639 48.3176)
-		(end 53.6918 56.2648)
+		(start 65.3364 45.7776)
+		(end 60.2224 45.7776)
 		(width 1.2)
 		(layer "B.Cu")
@@
 	)
 	(segment
+		(start 39.7764 29.464)
+		(end 69.088 29.464)
+		(width 1.2)
+		(layer "B.Cu")
+		(net 9)
+	)
+	(segment
+		(start 74.5744 34.9504)
+		(end 74.5744 40.7924)
+		(width 1.2)
+		(layer "B.Cu")
+		(net 9)
+	)
+	(segment
+		(start 36.6776 45.2628)
+		(end 36.6776 32.5628)
+		(width 1.2)
+		(layer "B.Cu")
+		(net 9)
+	)
+	(segment
+		(start 36.6776 32.5628)
+		(end 39.7764 29.464)
+		(width 1.2)
+		(layer "B.Cu")
+		(net 9)
+	)
+	(segment
+		(start 34.5186 47.4218)
+		(end 36.6776 45.2628)
+		(width 1.2)
+		(layer "B.Cu")
+		(net 9)
+	)
+	(segment
+		(start 31.0642 47.4218)
+		(end 34.5186 47.4218)
+		(width 1.2)
+		(layer "B.Cu")
+		(net 9)
+	)
+	(segment
+		(start 69.088 29.464)
+		(end 74.5744 34.9504)
+		(width 1.2)
+		(layer "B.Cu")
+		(net 9)
+	)
+	(segment
 		(start 31.0642 42.4218)
 		(end 27.1742 42.4218)
@@
 		(net 28)
 	)
-	(segment
-		(start 39.7764 29.464)
-		(end 69.088 29.464)
-		(width 1.2)
-		(layer "B.Cu")
-		(net 30)
-	)
-	(segment
-		(start 74.5744 34.9504)
-		(end 74.5744 40.7924)
-		(width 1.2)
-		(layer "B.Cu")
-		(net 30)
-	)
-	(segment
-		(start 36.6776 45.2628)
-		(end 36.6776 32.5628)
-		(width 1.2)
-		(layer "B.Cu")
-		(net 30)
-	)
-	(segment
-		(start 36.6776 32.5628)
-		(end 39.7764 29.464)
-		(width 1.2)
-		(layer "B.Cu")
-		(net 30)
-	)
-	(segment
-		(start 34.5186 47.4218)
-		(end 36.6776 45.2628)
-		(width 1.2)
-		(layer "B.Cu")
-		(net 30)
-	)
-	(segment
-		(start 31.0642 47.4218)
-		(end 34.5186 47.4218)
-		(width 1.2)
-		(layer "B.Cu")
-		(net 30)
-	)
-	(segment
-		(start 69.088 29.464)
-		(end 74.5744 34.9504)
-		(width 1.2)
-		(layer "B.Cu")
-		(net 30)
-	)
 )
